File: hardware/fc-board/mcu.kicad_sch (KiCad schematic)
At the start: 0 parts

Commit message: MCU sheet: F411 core, HSE, SWD, boot select; ERC fixes
Parts:
- added C20, C21, C22, C24, C25, C28: 100nF, Capacitor_SMD:C_0603_1608Metric, symbol Device:C
- added C23, C27: 4.7uF, Capacitor_SMD:C_0603_1608Metric, symbol Device:C
- added C26: 1uF, Capacitor_SMD:C_0603_1608Metric, symbol Device:C
- added C29, C30: 27pF, Capacitor_SMD:C_0603_1608Metric, symbol Device:C
- added FB1: 600R@100MHz, Inductor_SMD:L_0603_1608Metric, symbol Device:L
- added J2: SWD, Connector_PinHeader_2.54mm:PinHeader_1x04_P2.54mm_Vertical, symbol fc-board:Conn_01x04
- added J3: BOOT0_SEL, Connector_PinHeader_2.54mm:PinHeader_1x02_P2.54mm_Vertical, symbol Connector:Conn_01x02_Pin
- added R20, R21: 10k, Resistor_SMD:R_0603_1608Metric, symbol SparkFun-Resistor:10k_0603
- added U3: STM32F411CEU6, fc-board:UFQFPN-48_L7.0-W7.0-P0.50-BL-EP, symbol fc-board:STM32F411CEU6
- added Y1: 8MHz, Crystal:Crystal_SMD_5032-2Pin_5.0x3.2mm, symbol fc-board:Crystal
Connections:
- new net +3V3: C20.1, C21.1, C22.1, C23.1, C24.1, FB1.1, J2.3 (Pin_3), J3.1 (Pin_1), U3.1 (VBAT), U3.24 (VDD), U3.36 (VDD), U3.48 (VDD)
- new net BOOT0: J3.2 (Pin_2), R20.1, U3.44 (BOOT0)
- new net BOOT1: R21.1, U3.20 (PB2)
- new net GND: C20.2, C21.2, C22.2, C23.2, C24.2, C25.2, C26.2, C27.2, C28.2, C29.2, C30.2, J2.4 (Pin_4), R20.2, R21.2, U3.23 (VSS), U3.35 (VSS), U3.47 (VSS), U3.49 (PAD), U3.8 (VSSA/VREF-)
- new net HSE_IN: C29.1, U3.5 (PH0-OSC_IN), Y1.1
- new net HSE_OUT: C30.1, U3.6 (PH1-OSC_OUT), Y1.2
- new net IMU_CS: U3.14 (PA4)
- new net IMU_INT: U3.11 (PA1)
- new net IMU_MISO: U3.16 (PA6)
- new net IMU_MOSI: U3.17 (PA7)
- new net IMU_SCK: U3.15 (PA5)
- new net MOTOR1: U3.40 (PB4)
- new net MOTOR2: U3.41 (PB5)
- new net MOTOR3: U3.18 (PB0)
- new net MOTOR4: U3.19 (PB1)
- new net NRST: C28.1, U3.7 (NRST)
- new net RX_RX: U3.31 (PA10)
- new net RX_TX: U3.30 (PA9)
- new net SWCLK: J2.2 (Pin_2), U3.37 (PA14)
- new net SWDIO: J2.1 (Pin_1), U3.34 (PA13)
- new net USB_DM: U3.32 (PA11)
- new net USB_DP: U3.33 (PA12)
- new net VBAT_SENSE: U3.10 (PA0)
- new net VCAP1: C27.1, U3.22 (VCAP1)
- new net VDDA: C25.1, C26.1, FB1.2, U3.9 (VDDA/VREF+)
- no-connect marks 0 -> 17
Other:
- company: (none) -> Brody Barrett
- title: (none) -> STM32 Quadcopter Flight Controller
