File: hardware/fc-board/imu.kicad_sch (KiCad schematic)
At the start: 0 parts

Commit message: IMU sheet: ICM-42605 on SPI1
Parts:
- added C31: 100nF, Capacitor_SMD:C_0603_1608Metric, symbol Device:C
- added C32: 2.2uF, Capacitor_SMD:C_0603_1608Metric, symbol Device:C
- added C33: 10nF, Capacitor_SMD:C_0603_1608Metric, symbol Device:C
- added R22: 10k, Resistor_SMD:R_0603_1608Metric, symbol SparkFun-Resistor:10k_0603
- added U4: ICM-42605, fc-board:LGA-14_L3.0-W2.5-P0.50-TL, symbol fc-board:ICM-42605
Connections:
- new net +3V3: C31.1, C32.1, C33.1, R22.2, U4.5 (VDDIO), U4.8 (VDD)
- new net GND: C31.2, C32.2, C33.2, U4.6 (GND), U4.7 (RESV)
- new net IMU_CS: R22.1, U4.12 (AP_CS)
- new net IMU_INT: U4.4 (INT1/INT)
- new net IMU_MISO: U4.1 (AP_SDO/AP_AD0)
- new net IMU_MOSI: U4.14 (AP_SDA/AP_SDIO/AP_SDI)
- new net IMU_SCK: U4.13 (AP_SCL/AP_SCLK)
- no-connect marks 0 -> 5
Other:
- company: (none) -> Brody Barrett
- title: (none) -> STM32 Quadcopter Flight Controller
