File: hardware/fc-board/motors.kicad_sch (KiCad schematic)
At the start: 0 parts

Commit message: IMU, Motors, Radio sheets; schematic complete
Parts:
- added J4: ESC_SIGNAL, Connector_PinHeader_2.54mm:PinHeader_1x05_P2.54mm_Vertical, symbol fc-board:Conn_01x05
- added R23, R24, R25, R26: 33, Resistor_SMD:R_0603_1608Metric, symbol SparkFun-Resistor:R
Connections:
- new net: J4.1 (Pin_1), R23.2
- new net: J4.2 (Pin_2), R24.2
- new net: J4.3 (Pin_3), R25.2
- new net: J4.4 (Pin_4), R26.2
- new net GND: J4.5 (Pin_5)
- new net MOTOR1: R23.1
- new net MOTOR2: R24.1
- new net MOTOR3: R25.1
- new net MOTOR4: R26.1
Other:
- company: (none) -> Brody Barrett
- title: (none) -> STM32 Quadcopter Flight Controller
