File: hardware/fc-board/radio.kicad_sch (KiCad schematic)
At the start: 0 parts

Commit message: IMU, Motors, Radio sheets; schematic complete
Parts:
- added C34: 100nF, Capacitor_SMD:C_0603_1608Metric, symbol Device:C
- added C35: 10uF, Capacitor_SMD:C_0603_1608Metric, symbol Device:C
- added J5: ELRS_RX, Connector_PinHeader_2.54mm:PinHeader_1x04_P2.54mm_Vertical, symbol fc-board:Conn_01x04
Connections:
- new net +5V: C34.2, C35.2, J5.1 (Pin_1)
- new net GND: C34.1, C35.1, J5.2 (Pin_2)
- new net RX_RX: J5.3 (Pin_3)
- new net RX_TX: J5.4 (Pin_4)
Other:
- company: (none) -> Brody Barrett
- title: (none) -> STM32 Quadcopter Flight Controller
